Commit message: updating stretch.yml

File: resources/robot/stretchIsaac.urdf (robot description, URDF)
Before this commit: robot stretch, 44 links, 43 joints
Links:
- link base_imu: geometry collision mesh filename=meshes/base_imu.STL; visual mesh filename=meshes/base_imu.STL
- link base_link: geometry collision mesh filename=meshes/base_link.STL; visual mesh filename=meshes/base_link.STL
- link camera_link: geometry collision box size=0.02505 0.09 0.025; visual mesh filename=meshes/d435.dae
- link caster_link: geometry collision sphere radius=0.032; visual mesh filename=meshes/omni_wheel_m.STL
- link laser: geometry collision mesh filename=meshes/laser.STL; visual mesh filename=meshes/laser.STL
- link link_arm_l0: geometry collision mesh filename=meshes/link_arm_l0.STL; visual mesh filename=meshes/link_arm_l0.STL
- link link_arm_l1: geometry collision mesh filename=meshes/link_arm_l1.STL; visual mesh filename=meshes/link_arm_l1.STL
- link link_arm_l2: geometry collision mesh filename=meshes/link_arm_l2.STL; visual mesh filename=meshes/link_arm_l2.STL
- link link_arm_l3: geometry collision mesh filename=meshes/link_arm_l3.STL; visual mesh filename=meshes/link_arm_l3.STL
- link link_arm_l4: geometry collision mesh filename=meshes/link_arm_l4.STL; visual mesh filename=meshes/link_arm_l4.STL
- link link_aruco_inner_wrist: geometry collision mesh filename=meshes/link_aruco_inner_wrist.STL; visual mesh filename=meshes/link_aruco_inner_wrist.STL
- link link_aruco_left_base: geometry collision mesh filename=meshes/link_aruco_left_base.STL; visual mesh filename=meshes/link_aruco_left_base.STL
- link link_aruco_right_base: geometry collision mesh filename=meshes/link_aruco_right_base.STL; visual mesh filename=meshes/link_aruco_right_base.STL
- link link_aruco_shoulder: geometry collision mesh filename=meshes/link_aruco_shoulder.STL; visual mesh filename=meshes/link_aruco_shoulder.STL
- link link_aruco_top_wrist: geometry collision mesh filename=meshes/link_aruco_top_wrist.STL; visual mesh filename=meshes/link_aruco_top_wrist.STL
- link link_gripper: geometry collision mesh filename=meshes/link_gripper.STL; visual mesh filename=meshes/link_gripper.STL
- link link_gripper_finger_left: geometry collision mesh filename=meshes/link_gripper_finger_left.STL scale=0.9 1.0 1.0; visual mesh filename=meshes/link_gripper_finger_left.STL scale=0.9 1.0 1.0
- link link_gripper_finger_right: geometry collision mesh filename=meshes/link_gripper_finger_right.STL scale=0.9 1.0 1.0; visual mesh filename=meshes/link_gripper_finger_right.STL scale=0.9 1.0 1.0
- link link_gripper_fingertip_left: geometry collision mesh filename=meshes/link_gripper_fingertip_left.STL; visual mesh filename=meshes/link_gripper_fingertip_left.STL
- link link_gripper_fingertip_right: geometry collision mesh filename=meshes/link_gripper_fingertip_right.STL; visual mesh filename=meshes/link_gripper_fingertip_right.STL
- link link_head: geometry collision mesh filename=meshes/link_head.STL; visual mesh filename=meshes/link_head.STL
- link link_head_pan: geometry collision mesh filename=meshes/link_head_pan.STL; visual mesh filename=meshes/link_head_pan.STL
- link link_head_tilt: geometry collision mesh filename=meshes/link_head_tilt.STL; visual mesh filename=meshes/link_head_tilt.STL
- link link_left_wheel: geometry collision mesh filename=meshes/link_left_wheel.STL; visual mesh filename=meshes/link_left_wheel.STL
- link link_lift: geometry collision mesh filename=meshes/link_lift.STL; visual mesh filename=meshes/link_lift.STL
- link link_mast: geometry collision mesh filename=meshes/link_mast.STL; visual mesh filename=meshes/link_mast.STL
- link link_right_wheel: geometry collision mesh filename=meshes/link_right_wheel.STL; visual mesh filename=meshes/link_right_wheel.STL
- link link_wrist_yaw: geometry collision mesh filename=meshes/link_wrist_yaw.STL; visual mesh filename=meshes/link_wrist_yaw.STL
- link respeaker_base: geometry collision mesh filename=meshes/link_respeaker.STL; visual mesh filename=meshes/link_respeaker.STL
